File: trustflight_hardware.kicad_pcb (KiCad board)
At the start: 4 copper layers, 30.5 x 27 mm, 69 parts, among them J1 Conn_01x02, J10 Dronecode_Telemetry, J2 Conn_01x02, J3 Conn_01x02, J4 Conn_01x02, J5 Conn_01x01, J6 Conn_01x02, J7 Conn_01x02, J8 Conn_01x03, J9 swd-4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

Commit message: Updated silkscreen
Other:
- board text added: "5V"
- board text added: "Rev. B"
- board text removed: "+5V"
- board text removed: "Rev. A"
Changed lines of the file:
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@@
   (general
     (thickness 1.6)
-    (drawings 65)
+    (drawings 73)
     (tracks 741)
     (zones 0)
@@
     )
   )
+  (gr_line (start 148.3 100.8) (end 148.3 103.1) (layer B.SilkS) (width 0.3))
+  (gr_line (start 148.3 96.4) (end 148.3 100.8) (layer B.SilkS) (width 0.3))
+  (gr_line (start 143.9 95) (end 147.3 95) (layer B.SilkS) (width 0.3))
+  (gr_line (start 133 95) (end 133 100.5) (layer B.SilkS) (width 0.3))
+  (gr_line (start 143.9 95) (end 133 95) (layer B.SilkS) (width 0.3))
+  (gr_line (start 132.4 96.9) (end 126.9 96.9) (layer B.SilkS) (width 0.3))
+  (gr_line (start 132.4 82.7) (end 132.4 96.9) (layer B.SilkS) (width 0.3))
+  (gr_line (start 126.9 82.7) (end 132.4 82.7) (layer B.SilkS) (width 0.3))
   (gr_circle (center 147.7 102.3) (end 148 102.3) (layer F.SilkS) (width 0.4))
   (gr_text RC (at 129.8 96.1) (layer B.SilkS)
@@
     (effects (font (size 0.8 0.8) (thickness 0.2)))
   )
-  (gr_line (start 143.9 100.8) (end 147.8 100.8) (layer B.SilkS) (width 0.3))
-  (gr_line (start 143.9 95.6) (end 143.9 100.8) (layer B.SilkS) (width 0.3))
-  (gr_line (start 126.9 88.5) (end 131.3 88.5) (layer B.SilkS) (width 0.3))
+  (gr_line (start 143.9 100.8) (end 148.3 100.8) (layer B.SilkS) (width 0.3))
+  (gr_line (start 143.9 95) (end 143.9 100.8) (layer B.SilkS) (width 0.3))
+  (gr_line (start 126.9 88.5) (end 132.4 88.5) (layer B.SilkS) (width 0.3))
   (gr_text CERN-OHL (at 144.1 90.3 90) (layer B.SilkS)
     (effects (font (size 0.8 0.8) (thickness 0.2)) (justify mirror))
@@
   (gr_line (start 149 82) (end 149.5 83.5) (layer F.SilkS) (width 0.4))
   (gr_line (start 149 85) (end 152 83.5) (layer F.SilkS) (width 0.4))
-  (gr_text "Rev. A" (at 149 77.7) (layer B.SilkS)
+  (gr_text "Rev. B" (at 149 77.7) (layer B.SilkS)
     (effects (font (size 1 1) (thickness 0.25)) (justify mirror))
   )
-  (gr_text "Emil Fresk 2018" (at 149.1 84.7) (layer B.SilkS)
+  (gr_text "Emil Fresk 2018" (at 135.2 83.9 90) (layer B.SilkS)
     (effects (font (size 1 1) (thickness 0.25)) (justify mirror))
   )
-  (gr_text TrustFlight (at 150.1 82.7) (layer B.SilkS)
+  (gr_text TrustFlight (at 150.7 83.5) (layer B.SilkS)
     (effects (font (size 1.3 1.3) (thickness 0.3)) (justify mirror))
   )
@@
     (effects (font (size 0.8 0.8) (thickness 0.2)) (justify mirror))
   )
-  (gr_text GND (at 147.1 96.9 90) (layer B.SilkS)
+  (gr_text GND (at 147.3 96.9 90) (layer B.SilkS)
     (effects (font (size 0.8 0.8) (thickness 0.2)) (justify mirror))
   )
@@
     (effects (font (size 0.8 0.8) (thickness 0.2)) (justify mirror))
   )
-  (gr_text +5V (at 131.3 87) (layer B.SilkS)
+  (gr_text 5V (at 130.4 87) (layer B.SilkS)
     (effects (font (size 1.5 1.5) (thickness 0.3)) (justify mirror))
   )
